File: EdgeCubeH3/dram.kicad_sch (KiCad schematic)
At the start: 15 parts, among them U2 K4B4G1646Q

Commit message: Schematic update, PCB started
Parts:
- added C44: 1u, Capacitor_SMD:C_0603_1608Metric, symbol Device:C
- added U8: W25Q128JVP, Package_SON:WSON-8-1EP_6x5mm_P1.27mm_EP3.4x4.3mm, symbol Memory_Flash:W25Q128JVP
Connections:
- net GND: now also C44.2, U8.4 (GND), U8.9 (EP)
- new net +3V3: C44.1, U8.3 (~{WP}/IO_{2}), U8.7 (~{HOLD}/~{RESET}/IO_{3}), U8.8 (VCC)
- new net SPI0_CLK: U8.6 (CLK)
- new net SPI0_CS: U8.1 (~{CS})
- new net SPI0_MISO: U8.2 (DO/IO_{1})
- new net SPI0_MOSI: U8.5 (DI/IO_{0})
Other:
- note added: "NOR FLASH (OPTIONAL)"

Commit message: PCB design at ~90%
- re-arrangement of components
- connecting dram
- connecting ports
Parts:
- R5: footprint Resistor_SMD:R_0603_1608Metric -> Resistor_SMD:R_0402_1005Metric
Connections:
- net SDQ0: now also U2.F8 (DQ3); no longer U2.E3 (DQ0)
- net SDQ1: now also U2.H8 (DQ5); no longer U2.F7 (DQ1)
- net SDQ11: now also U2.D7 (DQ8); no longer U2.C2 (DQ11)
- net SDQ12: now also U2.A3 (DQ15); no longer U2.A7 (DQ12)
- net SDQ14: now also U2.C3 (DQ9); no longer U2.B8 (DQ14)
- net SDQ15: now also U2.C2 (DQ11); no longer U2.A3 (DQ15)
- net SDQ2: now also U2.F7 (DQ1); no longer U2.F2 (DQ2)
- net SDQ3: now also U2.G2 (DQ6); no longer U2.F8 (DQ3)
- net SDQ4: now also U2.H7 (DQ7); no longer U2.H3 (DQ4)
- net SDQ5: now also U2.E3 (DQ0); no longer U2.H8 (DQ5)
- net SDQ6: now also U2.F2 (DQ2); no longer U2.G2 (DQ6)
- net SDQ7: now also U2.H3 (DQ4); no longer U2.H7 (DQ7)
- net SDQ8: now also U2.A7 (DQ12); no longer U2.D7 (DQ8)
- net SDQ9: now also U2.B8 (DQ14); no longer U2.C3 (DQ9)
Changed lines of the file:
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@@
 	)
 	(label "SDQ2"
-		(at 179.07 49.53 180)
+		(at 179.07 46.99 180)
 		(effects
 			(font
@@
 	)
 	(label "SDQ3"
-		(at 179.07 52.07 180)
+		(at 179.07 59.69 180)
 		(effects
 			(font
@@
 	)
 	(label "SDQ1"
-		(at 179.07 46.99 180)
+		(at 179.07 57.15 180)
 		(effects
 			(font
@@
 	)
 	(label "SDQ0"
-		(at 179.07 44.45 180)
+		(at 179.07 52.07 180)
 		(effects
 			(font
@@
 	)
 	(label "SDQ9"
-		(at 179.07 67.31 180)
+		(at 179.07 80.01 180)
 		(effects
 			(font
@@
 	)
 	(label "SDQ11"
-		(at 179.07 72.39 180)
+		(at 179.07 64.77 180)
 		(effects
 			(font
@@
 	)
 	(label "SDQ7"
-		(at 179.07 62.23 180)
+		(at 179.07 54.61 180)
 		(effects
 			(font
@@
 	)
 	(label "SDQ5"
-		(at 179.07 57.15 180)
+		(at 179.07 44.45 180)
 		(effects
 			(font
@@
 	)
 	(label "SDQ12"
-		(at 179.07 74.93 180)
+		(at 179.07 82.55 180)
 		(effects
 			(font
@@
 	)
 	(label "SDQ6"
-		(at 179.07 59.69 180)
+		(at 179.07 49.53 180)
 		(effects
 			(font
@@
 	)
 	(label "SDQ15"
-		(at 179.07 82.55 180)
+		(at 179.07 72.39 180)
 		(effects
 			(font
@@
 	)
 	(label "SDQ8"
-		(at 179.07 64.77 180)
+		(at 179.07 74.93 180)
 		(effects
 			(font
@@
 	)
 	(label "SDQ14"
-		(at 179.07 80.01 180)
+		(at 179.07 67.31 180)
 		(effects
 			(font
@@
 	)
 	(label "SDQ4"
-		(at 179.07 54.61 180)
+		(at 179.07 62.23 180)
 		(effects
 			(font
@@
 			)
 		)
-		(property "Footprint" "Resistor_SMD:R_0603_1608Metric"
+		(property "Footprint" "Resistor_SMD:R_0402_1005Metric"
 			(at 187.96 154.178 90)
 			(hide yes)

Commit message: Compleating PCB design
Other:
- note added: "Termination under dram chip"
- moved on the sheet: R5
Changed lines of the file:
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@@
 		(company "github.com/sentoxo/EdgeCubeH3")
 	)
+	(text "Termination under dram chip"
+		(exclude_from_sim no)
+		(at 193.294 154.178 0)
+		(effects
+			(font
+				(size 1.27 1.27)
+			)
+		)
+	)
 	(text "NOR FLASH (OPTIONAL)"
 		(exclude_from_sim no)
@@
 	(wire
 		(pts
-			(xy 180.34 152.4) (xy 184.15 152.4)
+			(xy 185.42 151.13) (xy 189.23 151.13)
 		)
 		(stroke
@@
 	(wire
 		(pts
-			(xy 191.77 152.4) (xy 194.31 152.4)
+			(xy 196.85 151.13) (xy 199.39 151.13)
 		)
 		(stroke
@@
 	)
 	(label "SCK-"
-		(at 194.31 152.4 0)
+		(at 199.39 151.13 0)
 		(effects
 			(font
@@
 	)
 	(label "SCK+"
-		(at 180.34 152.4 180)
+		(at 185.42 151.13 180)
 		(effects
 			(font
@@
 	(symbol
 		(lib_id "Device:R")
-		(at 187.96 152.4 90)
+		(at 193.04 151.13 90)
 		(unit 1)
 		(body_style 1)
@@
 		(fields_autoplaced yes)
 		(property "Reference" "R5"
-			(at 187.96 146.05 90)
+			(at 193.04 144.78 90)
 			(show_name no)
 			(do_not_autoplace no)
@@
 		)
 		(property "Value" "100R"
-			(at 187.96 148.59 90)
+			(at 193.04 147.32 90)
 			(show_name no)
 			(do_not_autoplace no)
@@
 		)
 		(property "Footprint" "Resistor_SMD:R_0402_1005Metric"
-			(at 187.96 154.178 90)
+			(at 193.04 152.908 90)
 			(hide yes)
 			(show_name no)
@@
 		)
 		(property "Datasheet" ""
-			(at 187.96 152.4 0)
+			(at 193.04 151.13 0)
 			(hide yes)
 			(show_name no)
@@
 		)
 		(property "Description" "Resistor"
-			(at 187.96 152.4 0)
+			(at 193.04 151.13 0)
 			(hide yes)
 			(show_name no)
