File: EdgeCubeH3/power.kicad_sch (KiCad schematic)
At the start: 36 parts, among them J1 USB PWR, J2 SuperCap, Q1 NPN, Q2 PMOS, U3 USBLC6-2SC6, U5 SY8089AAAC, U6 SY8089AAAC, U7 SY8032

Commit message: Schematic update, PCB started
Parts:
- removed J2: SuperCap, Connector_PinHeader_2.54mm:PinHeader_1x02_P2.54mm_Vertical, symbol Connector:Conn_01x02_Socket
- added TP4: supercap, TestPoint:TestPoint_Pad_1.0x1.0mm, symbol Connector:TestPoint
- added TP5: gnd, TestPoint:TestPoint_Pad_1.0x1.0mm, symbol Connector:TestPoint
- C12, C15, C18: footprint Capacitor_SMD:C_0201_0603Metric -> Capacitor_SMD:C_0603_1608Metric
- Q1: footprint (none) -> Package_TO_SOT_SMD:TSOT-23
- Q2: footprint (none) -> Package_TO_SOT_SMD:SOT-23W
- R10, R11, R7, R8: footprint Resistor_SMD:R_0603_1608Metric_Pad0.98x0.95mm_HandSolder -> Capacitor_SMD:C_0603_1608Metric
- R12, R9: footprint Resistor_SMD:R_0805_2012Metric_Pad1.20x1.40mm_HandSolder -> Capacitor_SMD:C_0603_1608Metric
- R13, R14, R15, R16, R17, R18: footprint Resistor_SMD:R_0603_1608Metric_Pad0.98x0.95mm_HandSolder -> Resistor_SMD:R_0603_1608Metric
- U5, U6: footprint footprints:SY8089AAAC_SGY -> SY8089:SY8089AAAC_SGY
Connections:
- net GND: now also TP5.1
- net at D1.2 (A), R6.2: now also TP4.1
Other:
- moved on the sheet: R17, R18

Commit message: PCB design at ~90%
- re-arrangement of components
- connecting dram
- connecting ports
Parts:
- R19: footprint Resistor_SMD:R_0805_2012Metric_Pad1.20x1.40mm_HandSolder -> Resistor_SMD:R_0603_1608Metric_Pad0.98x0.95mm_HandSolder
Connections:
- net USB+: now reaches J1.A6 (D+), J1.B6 (D+), U3.3 (I/O2)
- net USB-: now reaches J1.A7 (D-), J1.B7 (D-), U3.1 (I/O1)
Other:
- moved on the sheet: U3
Changed lines of the file:
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@@
 	)
 	(junction
-		(at 181.61 49.53)
+		(at 53.34 46.99)
 		(diameter 0)
 		(color 0 0 0 0)
 	)
 	(junction
-		(at 106.68 135.89)
+		(at 181.61 49.53)
 		(diameter 0)
 		(color 0 0 0 0)
 	)
 	(junction
-		(at 77.47 31.75)
+		(at 106.68 135.89)
 		(diameter 0)
 		(color 0 0 0 0)
 	)
 	(junction
-		(at 53.34 46.99)
+		(at 77.47 31.75)
 		(diameter 0)
 		(color 0 0 0 0)
@@
 	)
 	(junction
-		(at 53.34 49.53)
-		(diameter 0)
-		(color 0 0 0 0)
-	)
-	(junction
 		(at 180.34 90.17)
 		(diameter 0)
@@
 	)
 	(junction
+		(at 53.34 49.53)
+		(diameter 0)
+		(color 0 0 0 0)
+	)
+	(junction
 		(at 33.02 121.92)
 		(diameter 0)
@@
 	)
 	(junction
+		(at 63.5 31.75)
+		(diameter 0)
+		(color 0 0 0 0)
+	)
+	(junction
 		(at 255.27 35.56)
 		(diameter 0)
@@
 	(wire
 		(pts
+			(xy 63.5 31.75) (xy 68.58 31.75)
+		)
+		(stroke
+			(width 0)
+			(type default)
+		)
+	)
+	(wire
+		(pts
 			(xy 173.99 41.91) (xy 181.61 41.91)
 		)
@@
 	(wire
 		(pts
+			(xy 63.5 31.75) (xy 62.23 31.75)
+		)
+		(stroke
+			(width 0)
+			(type default)
+		)
+	)
+	(wire
+		(pts
 			(xy 180.34 90.17) (xy 190.5 90.17)
 		)
@@
 	(wire
 		(pts
-			(xy 57.15 49.53) (xy 53.34 49.53)
+			(xy 58.42 49.53) (xy 53.34 49.53)
 		)
 		(stroke
@@
 	(wire
 		(pts
-			(xy 67.31 49.53) (xy 76.2 49.53)
+			(xy 68.58 49.53) (xy 76.2 49.53)
 		)
 		(stroke
@@
 	(wire
 		(pts
-			(xy 62.23 31.75) (xy 68.58 31.75)
-		)
-		(stroke
-			(width 0)
-			(type default)
-		)
-	)
-	(wire
-		(pts
 			(xy 105.41 82.55) (xy 105.41 83.82)
 		)
@@
 	(wire
 		(pts
-			(xy 62.23 69.85) (xy 38.1 69.85)
+			(xy 63.5 69.85) (xy 38.1 69.85)
 		)
 		(stroke
@@
 	(wire
 		(pts
-			(xy 62.23 31.75) (xy 62.23 41.91)
+			(xy 63.5 31.75) (xy 63.5 41.91)
 		)
 		(stroke
@@
 	(wire
 		(pts
-			(xy 67.31 46.99) (xy 76.2 46.99)
+			(xy 68.58 46.99) (xy 76.2 46.99)
 		)
 		(stroke
@@
 	(wire
 		(pts
-			(xy 62.23 54.61) (xy 62.23 69.85)
+			(xy 63.5 54.61) (xy 63.5 69.85)
 		)
 		(stroke
@@
 	(wire
 		(pts
-			(xy 57.15 46.99) (xy 53.34 46.99)
+			(xy 58.42 46.99) (xy 53.34 46.99)
 		)
 		(stroke
@@
 		)
 	)
+	(label "USB-"
+		(at 53.34 46.99 0)
+		(effects
+			(font
+				(size 1.27 1.27)
+			)
+			(justify left bottom)
+		)
+	)
+	(label "USB+"
+		(at 53.34 49.53 0)
+		(effects
+			(font
+				(size 1.27 1.27)
+			)
+			(justify left bottom)
+		)
+	)
 	(global_label "PWR_DRAM_EN"
 		(shape input)
@@
 			)
 		)
-		(property "Footprint" "Resistor_SMD:R_0805_2012Metric_Pad1.20x1.40mm_HandSolder"
+		(property "Footprint" "Resistor_SMD:R_0603_1608Metric_Pad0.98x0.95mm_HandSolder"
 			(at 249.682 45.72 90)
 			(hide yes)
@@
 	(symbol
 		(lib_id "Power_Protection:USBLC6-2SC6")
-		(at 62.23 46.99 0)
+		(at 63.5 46.99 0)
 		(unit 1)
 		(body_style 1)
@@
 		(dnp no)
 		(property "Reference" "U3"
-			(at 62.992 42.672 0)
+			(at 64.262 42.672 0)
 			(show_name no)
 			(do_not_autoplace no)
@@
 		)
 		(property "Value" "USBLC6-2SC6"
-			(at 62.992 54.102 0)
+			(at 64.262 54.102 0)
 			(show_name no)
 			(do_not_autoplace no)
@@
 		)
 		(property "Footprint" "Package_TO_SOT_SMD:SOT-23-6"
-			(at 63.5 53.34 0)
+			(at 64.77 53.34 0)
 			(hide yes)
 			(show_name no)
@@
 		)
 		(property "Datasheet" "https://www.st.com/resource/en/datasheet/usblc6-2.pdf"
-			(at 63.5 55.245 0)
+			(at 64.77 55.245 0)
 			(hide yes)
 			(show_name no)
@@
 		)
 		(property "Description" "Very low capacitance ESD protection diode, 2 data-line, SOT-23-6"
-			(at 62.23 46.99 0)
+			(at 63.5 46.99 0)
 			(hide yes)
 			(show_name no)

Commit message: Small changes to PCB, updated schematic and readme
Parts:
- added R48, R49: 5K1, Capacitor_SMD:C_0603_1608Metric, symbol Device:R
Connections:
- net GND: now also R48.2, R49.1
- net at J1.A5 (CC1): now also R48.1
- net at J1.B5 (CC2): now also R49.2
- no-connect marks 5 -> 3
Changed lines of the file:
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@@
 	(title_block
 		(title "EdgeCubeH3")
-		(date "2026-05-07")
-		(rev "0.1")
+		(date "2026-05-21")
+		(rev "rev.A")
 		(company "github.com/sentoxo/EdgeCubeH3")
 	)
@@
 	)
 	(junction
+		(at 68.58 39.37)
+		(diameter 0)
+		(color 0 0 0 0)
+	)
+	(junction
 		(at 106.68 128.27)
 		(diameter 0)
@@
 	)
 	(junction
+		(at 60.96 39.37)
+		(diameter 0)
+		(color 0 0 0 0)
+	)
+	(junction
 		(at 255.27 35.56)
 		(diameter 0)
@@
 	)
 	(no_connect
-		(at 53.34 39.37)
-	)
-	(no_connect
 		(at 53.34 62.23)
 	)
-	(no_connect
-		(at 53.34 36.83)
-	)
 	(wire
 		(pts
@@
 	(wire
 		(pts
+			(xy 60.96 36.83) (xy 60.96 39.37)
+		)
+		(stroke
+			(width 0)
+			(type default)
+		)
+	)
+	(wire
+		(pts
 			(xy 53.34 44.45) (xy 53.34 46.99)
 		)
@@
 	(wire
 		(pts
+			(xy 60.96 39.37) (xy 68.58 39.37)
+		)
+		(stroke
+			(width 0)
+			(type default)
+		)
+	)
+	(wire
+		(pts
 			(xy 167.64 90.17) (xy 170.18 90.17)
 		)
@@
 	)
 	(symbol
+		(lib_id "Device:R")
+		(at 57.15 36.83 90)
+		(unit 1)
+		(body_style 1)
+		(exclude_from_sim no)
+		(in_bom yes)
+		(on_board yes)
+		(in_pos_files yes)
+		(dnp no)
+		(property "Reference" "R48"
+			(at 57.15 34.798 90)
+			(show_name no)
+			(do_not_autoplace no)
+			(effects
+				(font
+					(size 1.27 1.27)
+				)
+			)
+		)
+		(property "Value" "5K1"
+			(at 57.15 36.83 90)
+			(show_name no)
+			(do_not_autoplace no)
+			(effects
+				(font
+					(size 1.27 1.27)
+				)
+			)
+		)
+		(property "Footprint" "Capacitor_SMD:C_0603_1608Metric"
+			(at 57.15 38.608 90)
+			(hide yes)
+			(show_name no)
+			(do_not_autoplace no)
+			(effects
+				(font
+					(size 1.27 1.27)
+				)
+			)
+		)
+		(property "Datasheet" ""
+			(at 57.15 36.83 0)
+			(hide yes)
+			(show_name no)
+			(do_not_autoplace no)
+			(effects
+				(font
+					(size 1.27 1.27)
+				)
+			)
+		)
+		(property "Description" "Resistor"
+			(at 57.15 36.83 0)
+			(hide yes)
+			(show_name no)
+			(do_not_autoplace no)
+			(effects
+				(font
+					(size 1.27 1.27)
+				)
+			)
+		)
+		(pin "2"
+		)
+		(pin "1"
+		)
+		(instances
+			(project "EdgeCubeH3"
+				(path "/36b001b0-3d06-4fed-b406-d82b909f7864/91a9e285-5308-4a22-be4b-5a32b9b39521"
+					(reference "R48")
+					(unit 1)
+				)
+			)
+		)
+	)
+	(symbol
 		(lib_id "power:GND")
 		(at 116.84 91.44 0)
@@
 					(unit 1)
 				)
+			)
+		)
+	)
+	(symbol
+		(lib_id "Device:R")
+		(at 57.15 39.37 270)
+		(unit 1)
+		(body_style 1)
+		(exclude_from_sim no)
+		(in_bom yes)
+		(on_board yes)
+		(in_pos_files yes)
+		(dnp no)
+		(property "Reference" "R49"
+			(at 57.15 41.402 90)
+			(show_name no)
+			(do_not_autoplace no)
+			(effects
+				(font
+					(size 1.27 1.27)
+				)
+			)
+		)
+		(property "Value" "5K1"
+			(at 57.15 39.37 90)
+			(show_name no)
+			(do_not_autoplace no)
+			(effects
+				(font
+					(size 1.27 1.27)
+				)
+			)
+		)
+		(property "Footprint" "Capacitor_SMD:C_0603_1608Metric"
+			(at 57.15 37.592 90)
+			(hide yes)
+			(show_name no)
+			(do_not_autoplace no)
+			(effects
+				(font
+					(size 1.27 1.27)
+				)
+			)
+		)
+		(property "Datasheet" ""
+			(at 57.15 39.37 0)
+			(hide yes)
+			(show_name no)
+			(do_not_autoplace no)
+			(effects
+				(font
+					(size 1.27 1.27)
+				)
+			)
+		)
+		(property "Description" "Resistor"
+			(at 57.15 39.37 0)
+			(hide yes)
+			(show_name no)
+			(do_not_autoplace no)
+			(effects
+				(font
+					(size 1.27 1.27)
+				)
+			)
+		)
+		(pin "2"
+		)
+		(pin "1"
+		)
+		(instances
+			(project "EdgeCubeH3"
+				(path "/36b001b0-3d06-4fed-b406-d82b909f7864/91a9e285-5308-4a22-be4b-5a32b9b39521"
+					(reference "R49")
+					(unit 1)
+				)

Commit message: Finalization of rev.A
Parts:
- removed TP4: supercap, TestPoint:TestPoint_Pad_1.0x1.0mm, symbol Connector:TestPoint
- removed TP5: gnd, TestPoint:TestPoint_Pad_1.0x1.0mm, symbol Connector:TestPoint
- added J2: SUPERCAP, Connector_PinHeader_1.27mm:PinHeader_1x02_P1.27mm_Vertical, symbol Connector:Conn_01x02_Pin
- R48, R49: footprint Capacitor_SMD:C_0603_1608Metric -> Resistor_SMD:R_0603_1608Metric; now not fitted
Connections:
- net GND: now also J2.1 (Pin_1)
- net at D1.2 (A), R6.2: now also J2.2 (Pin_2)
Changed lines of the file:
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@@
 	)
 	(symbol
-		(lib_id "Connector:TestPoint")
-		(at 88.9 31.75 270)
+		(lib_id "Connector:Conn_01x02_Pin")
+		(at 93.98 34.29 180)
 		(unit 1)
 		(body_style 1)
@@
 		(dnp no)
 		(fields_autoplaced yes)
-		(property "Reference" "TP4"
-			(at 93.98 30.4799 90)
+		(property "Reference" "J2"
+			(at 95.25 31.7499 0)
 			(show_name no)
 			(do_not_autoplace no)
@@
 					(size 1.27 1.27)
 				)
-				(justify left)
+				(justify right)
 			)
 		)
-		(property "Value" "supercap"
-			(at 93.98 33.0199 90)
+		(property "Value" "SUPERCAP"
+			(at 95.25 34.2899 0)
 			(show_name no)
 			(do_not_autoplace no)
@@
 					(size 1.27 1.27)
 				)
-				(justify left)
+				(justify right)
 			)
 		)
-		(property "Footprint" "TestPoint:TestPoint_Pad_1.0x1.0mm"
-			(at 88.9 36.83 0)
+		(property "Footprint" "Connector_PinHeader_1.27mm:PinHeader_1x02_P1.27mm_Vertical"
+			(at 93.98 34.29 0)
 			(hide yes)
 			(show_name no)
@@
 		)
 		(property "Datasheet" ""
-			(at 88.9 36.83 0)
+			(at 93.98 34.29 0)
 			(hide yes)
 			(show_name no)
@@
 			)
 		)
-		(property "Description" "test point"
-			(at 88.9 31.75 0)
+		(property "Description" "Generic connector, single row, 01x02, script generated"
+			(at 93.98 34.29 0)
 			(hide yes)
 			(show_name no)
@@
 			)
 		)
+		(pin "2"
+		)
 		(pin "1"
 		)
@@
 			(project "EdgeCubeH3"
 				(path "/36b001b0-3d06-4fed-b406-d82b909f7864/91a9e285-5308-4a22-be4b-5a32b9b39521"
-					(reference "TP4")
+					(reference "J2")
 					(unit 1)
 				)
@@
 	(symbol
 		(lib_id "power:GND")
-		(at 88.9 36.83 0)
+		(at 88.9 34.29 0)
 		(unit 1)
 		(body_style 1)
@@
 		(dnp no)
 		(property "Reference" "#PWR015"
-			(at 88.9 43.18 0)
+			(at 88.9 40.64 0)
 			(hide yes)
 			(show_name no)
@@
 		)
 		(property "Value" "GND"
-			(at 88.9 40.64 0)
+			(at 88.9 38.1 0)
 			(show_name no)
 			(do_not_autoplace no)
@@
 		)
 		(property "Footprint" ""
-			(at 88.9 36.83 0)
+			(at 88.9 34.29 0)
 			(hide yes)
 			(show_name no)
@@
 		)
 		(property "Datasheet" ""
-			(at 88.9 36.83 0)
+			(at 88.9 34.29 0)
 			(hide yes)
 			(show_name no)
@@
 		)
 		(property "Description" "Power symbol creates a global label with name \"GND\" , ground"
-			(at 88.9 36.83 0)
+			(at 88.9 34.29 0)
 			(hide yes)
 			(show_name no)
@@
 	)
 	(symbol
-		(lib_id "Connector:TestPoint")
-		(at 88.9 36.83 270)
-		(unit 1)
-		(body_style 1)
-		(exclude_from_sim no)
-		(in_bom yes)
-		(on_board yes)
-		(in_pos_files yes)
-		(dnp no)
-		(fields_autoplaced yes)
-		(property "Reference" "TP5"
-			(at 93.98 35.5599 90)
-			(show_name no)
-			(do_not_autoplace no)
-			(effects
-				(font
-					(size 1.27 1.27)
-				)
-				(justify left)
-			)
-		)
-		(property "Value" "gnd"
-			(at 93.98 38.0999 90)
-			(show_name no)
-			(do_not_autoplace no)
-			(effects
-				(font
-					(size 1.27 1.27)
-				)
-				(justify left)
-			)
-		)
-		(property "Footprint" "TestPoint:TestPoint_Pad_1.0x1.0mm"
-			(at 88.9 41.91 0)
-			(hide yes)
-			(show_name no)
-			(do_not_autoplace no)
-			(effects
-				(font
-					(size 1.27 1.27)
-				)
-			)
-		)
-		(property "Datasheet" ""
-			(at 88.9 41.91 0)
-			(hide yes)
-			(show_name no)
-			(do_not_autoplace no)
-			(effects
-				(font
-					(size 1.27 1.27)
-				)
-			)
-		)
-		(property "Description" "test point"
-			(at 88.9 36.83 0)
-			(hide yes)
-			(show_name no)
-			(do_not_autoplace no)
-			(effects
-				(font
-					(size 1.27 1.27)
-				)
-			)
-		)
-		(pin "1"
-		)
-		(instances
-			(project "EdgeCubeH3"
-				(path "/36b001b0-3d06-4fed-b406-d82b909f7864/91a9e285-5308-4a22-be4b-5a32b9b39521"
-					(reference "TP5")
-					(unit 1)
-				)
-			)
-		)
-	)
-	(symbol
 		(lib_id "power:PWR_FLAG")
 		(at 172.72 90.17 0)
@@
 		(on_board yes)
 		(in_pos_files yes)
-		(dnp no)
+		(dnp yes)
 		(property "Reference" "R48"
 			(at 57.15 34.798 90)
@@
 			)
 		)
-		(property "Footprint" "Capacitor_SMD:C_0603_1608Metric"
+		(property "Footprint" "Resistor_SMD:R_0603_1608Metric"
 			(at 57.15 38.608 90)
 			(hide yes)
@@
 		(on_board yes)
 		(in_pos_files yes)
-		(dnp no)
+		(dnp yes)
 		(property "Reference" "R49"
 			(at 57.15 41.402 90)
@@
 			)
 		)
-		(property "Footprint" "Capacitor_SMD:C_0603_1608Metric"
+		(property "Footprint" "Resistor_SMD:R_0603_1608Metric"
 			(at 57.15 37.592 90)
 			(hide yes)
